Commit message: Migrate from _gripper postfix to directly use rv2fr

File: melfa_description/urdf/rv2fr/rv2fr.urdf.xacro (robot description, xacro)
@@ -2,6 +2,6 @@
 <robot xmlns:xacro="http://www.ros.org/wiki/xacro" name="rv2fr">
     <!-- Enable setting arguments from the launch file -->
-    <xacro:arg name="use_sim" default="false" />
-    <xacro:arg name="use_fake_hardware" default="true" />
+    <xacro:arg name="use_sim" default="true" />
+    <xacro:arg name="use_fake_hardware" default="false" />
     <xacro:arg name="prefix" default="" />
     <xacro:arg name="robot_ip" default="192.168.0.20" />
@@ -17,13 +17,39 @@
     <xacro:arg name="packet_lost_log" default="1" />
     <xacro:arg name="simulation_controllers" default="" />
+    <!-- Include the gripper settings -->
+    <xacro:arg name="sim_gazebo" default="$(arg use_sim)" />
+    <xacro:arg name="use_mock_hardware" default="$(arg use_fake_hardware)" />
+    <!-- After your existing arguments, before the include -->
     <!-- Import urdf file -->
+    <!-- Here we include a macro file, so later we still need to call the macro to spawn the manipulator -->
     <xacro:include filename="$(find melfa_description)/urdf/rv2fr/rv2fr_macro.xacro" />
     <!-- Import ros2_control description -->
+    <!-- Here this xacro file is actually a macro file, so later we still need to call the macro -->
     <xacro:include filename="$(find melfa_description)/ros2_control/rv2fr.hardware.xacro" />
     <!-- Use world link to fix robot -->
     <link name="$(arg prefix)world"/>
+    <!-- Spawn the manipulator -->
     <xacro:rv2fr parent="$(arg prefix)world" prefix="$(arg prefix)">
         <origin xyz="0 0 0" rpy="0 0 0" />
     </xacro:rv2fr>
+    <!-- Import robotiq_hand_e_gripper -->
+    <!-- Here this file is a xacro, in it it calls macro to spawn the gripper -->
+    <!-- Use this if parameters are set from the launch file, otherwise delete -->
+    <xacro:arg name="parent" default="$(arg prefix)rv2fr_default_tcp" />
+    <xacro:arg name="mock_sensor_commands" default="false" />
+    <xacro:include filename="$(find robotiq_description)/urdf/robotiq_hand_e_macro.urdf.xacro"/>
+    <xacro:include filename="$(find robotiq_description)/urdf/hand_e.ros2_control.xacro"/>
+    <!-- create link fixed to the "world" -->
+    <!-- <link name="base_link" /> -->
+    <!-- Load robot's macro with parameters -->
+    <!-- set prefix if multiple robots are used -->
+    <xacro:robotiq_hande prefix="$(arg prefix)" parent="$(arg parent)">
+        <origin xyz="0 0 0" rpy="0 0 0" />
+    </xacro:robotiq_hande>
+    <xacro:robotiq_hande_ros2_control
+        name="robotiq_hande"
+        prefix="$(arg prefix)"
+        sim_gazebo="$(arg sim_gazebo)"
+        use_mock_hardware="$(arg use_mock_hardware)" />
     <xacro:rv2fr_hardware
         name="rv2fr"
@@ -42,5 +68,15 @@
         controller_type="$(arg controller_type)"
         packet_lost_log="$(arg packet_lost_log)"
-        />
+    />
+    <!-- <xacro:if value="$(arg use_sim)">
+        <gazebo reference="world">
+        </gazebo>
+        <gazebo>
+        <plugin filename="gz_ros2_control-system" name="gz_ros2_control::GazeboSimROS2ControlPlugin">
+            <parameters>$(arg simulation_controllers)</parameters>
+            <controller_manager_node_name>$(arg prefix)controller_manager</controller_manager_node_name>
+        </plugin>
+        </gazebo>
+    </xacro:if> -->
     <xacro:if value="$(arg use_sim)">
         <!-- Gazebo plugins -->
@@ -48,8 +84,8 @@
         </gazebo>
         <gazebo>
-        <plugin filename="libign_ros2_control-system.so" name="ign_ros2_control::IgnitionROS2ControlPlugin">
-            <parameters>$(arg simulation_controllers)</parameters>
-            <controller_manager_node_name>$(arg prefix)controller_manager</controller_manager_node_name>
-        </plugin>
+            <plugin filename="ign_ros2_control-system" name="ign_ros2_control::IgnitionROS2ControlPlugin">
+                <parameters>$(arg simulation_controllers)</parameters>
+                <controller_manager_node_name>$(arg prefix)controller_manager</controller_manager_node_name>
+            </plugin>
         </gazebo>
     </xacro:if>

File: melfa_moveit_config/melfa_rv2fr_moveit_config/config/rv2fr_macro.srdf.xacro (robot description, xacro)
@@ -11,15 +11,17 @@
         <!--CHAINS: When a chain is specified, all the links along the chain (including endpoints) are included in the group. Additionally, all the joints that are parents to included links are also included. This means that joints along the chain and the parent joint of the base link are included in the group-->
         <!--SUBGROUPS: Groups can also be formed by referencing to already defined group names-->
-       <group name="rv2fr">
-        <joint name="rv2fr_joint_1"/>
-        <joint name="rv2fr_joint_2"/>
-        <joint name="rv2fr_joint_3"/>
-        <joint name="rv2fr_joint_4"/>
-        <joint name="rv2fr_joint_5"/>
-        <joint name="rv2fr_joint_6"/>
-        <joint name="rv2fr_hand_tcp"/>
-        <chain base_link="rv2fr_base" tip_link="rv2fr_default_tcp"/>
+        <!-- Main robot arm group -->
+        <group name="rv2fr">
+            <joint name="rv2fr_joint_1"/>
+            <joint name="rv2fr_joint_2"/>
+            <joint name="rv2fr_joint_3"/>
+            <joint name="rv2fr_joint_4"/>
+            <joint name="rv2fr_joint_5"/>
+            <joint name="rv2fr_joint_6"/>
+            <joint name="rv2fr_hand_tcp"/>
+            <chain base_link="rv2fr_base" tip_link="tcp_link"/>
         </group>
         <!--GROUP STATES: Purpose: Define a named state for a particular group, in terms of joint values. This is useful to define states like 'folded arms'-->
+        <!-- Original arm positions -->
         <group_state name="home" group="rv2fr">
             <joint name="rv2fr_joint_1" value="0"/>
@@ -30,13 +32,6 @@
             <joint name="rv2fr_joint_6" value="0"/>
         </group_state>
-        <group_state name="home_tool" group="rv2fr">
-            <joint name="rv2fr_joint_1" value="0"/>
-            <joint name="rv2fr_joint_2" value="0"/>
-            <joint name="rv2fr_joint_3" value="1.5708"/>
-            <joint name="rv2fr_joint_4" value="0"/>
-            <joint name="rv2fr_joint_5" value="-1.5708"/>
-            <joint name="rv2fr_joint_6" value="0"/>
-        </group_state>
         <!--DISABLE COLLISIONS: By default it is assumed that any link of the robot could potentially come into collision with any other link in the robot. This tag disables collision checking between a specified pair of links. -->
+        <!-- Original robot arm collision disabling -->
         <disable_collisions link1="rv2fr_base" link2="rv2fr_shoulder" reason="Adjacent"/>
         <disable_collisions link1="rv2fr_base" link2="rv2fr_upper_arm" reason="Never"/>
@@ -53,4 +48,70 @@
         <disable_collisions link1="rv2fr_shoulder" link2="rv2fr_upper_arm" reason="Adjacent"/>
         <disable_collisions link1="rv2fr_upper_arm" link2="rv2fr_wrist" reason="Never"/>
+        <disable_collisions link1="rv2fr_base" link2="rv2fr_default_tcp" reason="Never"/>
+        <disable_collisions link1="rv2fr_base" link2="hand_e_base_link" reason="Never"/>
+        <disable_collisions link1="rv2fr_base" link2="hande_finger_distance_link" reason="Never"/>
+        <disable_collisions link1="rv2fr_base" link2="hande_left_finger" reason="Never"/>
+        <disable_collisions link1="rv2fr_base" link2="hande_right_finger" reason="Never"/>
+        <disable_collisions link1="rv2fr_base" link2="tcp_link" reason="Never"/>
+        <disable_collisions link1="rv2fr_shoulder" link2="rv2fr_default_tcp" reason="Never"/>
+        <disable_collisions link1="rv2fr_shoulder" link2="hand_e_base_link" reason="Never"/>
+        <disable_collisions link1="rv2fr_shoulder" link2="hande_finger_distance_link" reason="Never"/>
+        <disable_collisions link1="rv2fr_shoulder" link2="hande_left_finger" reason="Never"/>
+        <disable_collisions link1="rv2fr_shoulder" link2="hande_right_finger" reason="Never"/>
+        <disable_collisions link1="rv2fr_shoulder" link2="tcp_link" reason="Never"/>
+        <!-- Gripper internal collision disabling -->
+        <disable_collisions link1="hand_e_base_link" link2="hande_finger_distance_link" reason="Adjacent"/>
+        <disable_collisions link1="hand_e_base_link" link2="hande_left_finger" reason="Adjacent"/>
+        <disable_collisions link1="hand_e_base_link" link2="hande_right_finger" reason="Adjacent"/>
+        <disable_collisions link1="hande_left_finger" link2="hande_right_finger" reason="Never"/>
+        <disable_collisions link1="hande_left_finger" link2="hande_finger_distance_link" reason="Never"/>
+        <disable_collisions link1="hande_right_finger" link2="hande_finger_distance_link" reason="Never"/>
+        <!-- Gripper to arm collision disabling - direct connections -->
+        <disable_collisions link1="rv2fr_hand_flange" link2="rv2fr_default_tcp" reason="Adjacent"/>
+        <disable_collisions link1="rv2fr_default_tcp" link2="hand_e_base_link" reason="Adjacent"/>
+        <!-- Wrist to gripper -->
+        <disable_collisions link1="rv2fr_wrist" link2="rv2fr_default_tcp" reason="Never"/>
+        <disable_collisions link1="rv2fr_wrist" link2="hand_e_base_link" reason="Never"/>
+        <disable_collisions link1="rv2fr_wrist" link2="hande_finger_distance_link" reason="Never"/>
+        <disable_collisions link1="rv2fr_wrist" link2="hande_left_finger" reason="Never"/>
+        <disable_collisions link1="rv2fr_wrist" link2="hande_right_finger" reason="Never"/>
+        <disable_collisions link1="rv2fr_wrist" link2="tcp_link" reason="Never"/>
+        <!-- Hand flange to gripper components -->
+        <disable_collisions link1="rv2fr_hand_flange" link2="hand_e_base_link" reason="Never"/>
+        <disable_collisions link1="rv2fr_hand_flange" link2="hande_finger_distance_link" reason="Never"/>
+        <disable_collisions link1="rv2fr_hand_flange" link2="hande_left_finger" reason="Never"/>
+        <disable_collisions link1="rv2fr_hand_flange" link2="hande_right_finger" reason="Never"/>
+        <disable_collisions link1="rv2fr_hand_flange" link2="tcp_link" reason="Never"/>
+        <!-- Default TCP to gripper -->
+        <disable_collisions link1="rv2fr_default_tcp" link2="hande_finger_distance_link" reason="Never"/>
+        <disable_collisions link1="rv2fr_default_tcp" link2="hande_left_finger" reason="Never"/>
+        <disable_collisions link1="rv2fr_default_tcp" link2="hande_right_finger" reason="Never"/>
+        <disable_collisions link1="rv2fr_default_tcp" link2="tcp_link" reason="Never"/>
+        <!-- Forearm to gripper -->
+        <disable_collisions link1="rv2fr_forearm" link2="rv2fr_default_tcp" reason="Never"/>
+        <disable_collisions link1="rv2fr_forearm" link2="hand_e_base_link" reason="Never"/>
+        <disable_collisions link1="rv2fr_forearm" link2="hande_finger_distance_link" reason="Never"/>
+        <disable_collisions link1="rv2fr_forearm" link2="hande_left_finger" reason="Never"/>
+        <disable_collisions link1="rv2fr_forearm" link2="hande_right_finger" reason="Never"/>
+        <disable_collisions link1="rv2fr_forearm" link2="tcp_link" reason="Never"/>
+        <!-- Elbow to gripper -->
+        <disable_collisions link1="rv2fr_elbow" link2="rv2fr_default_tcp" reason="Never"/>
+        <disable_collisions link1="rv2fr_elbow" link2="hand_e_base_link" reason="Never"/>
+        <disable_collisions link1="rv2fr_elbow" link2="hande_finger_distance_link" reason="Never"/>
+        <disable_collisions link1="rv2fr_elbow" link2="hande_left_finger" reason="Never"/>
+        <disable_collisions link1="rv2fr_elbow" link2="hande_right_finger" reason="Never"/>
+        <disable_collisions link1="rv2fr_elbow" link2="tcp_link" reason="Never"/>
+        <!-- Upper arm to gripper -->
+        <disable_collisions link1="rv2fr_upper_arm" link2="rv2fr_default_tcp" reason="Never"/>
+        <disable_collisions link1="rv2fr_upper_arm" link2="hand_e_base_link" reason="Never"/>
+        <disable_collisions link1="rv2fr_upper_arm" link2="hande_finger_distance_link" reason="Never"/>
+        <disable_collisions link1="rv2fr_upper_arm" link2="hande_left_finger" reason="Never"/>
+        <disable_collisions link1="rv2fr_upper_arm" link2="hande_right_finger" reason="Never"/>
+        <disable_collisions link1="rv2fr_upper_arm" link2="tcp_link" reason="Never"/>
+        <!-- TCP link connections -->
+        <disable_collisions link1="hand_e_base_link" link2="tcp_link" reason="Adjacent"/>
+        <disable_collisions link1="hande_finger_distance_link" link2="tcp_link" reason="Never"/>
+        <disable_collisions link1="hande_left_finger" link2="tcp_link" reason="Never"/>
+        <disable_collisions link1="hande_right_finger" link2="tcp_link" reason="Never"/>
     </xacro:macro>
 </robot>
