Commit message: Update configs for moveit pkg.

File: melfa_description/urdf/rv2fr/rv2fr.urdf (robot description, URDF)
Before this commit: robot rv2fr, 9 links, 8 joints
Links:
- added link hand_e_base_link; collision mesh filename=package://robotiq_description/meshes/collision/hande/hand-e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 scale=1.0 1.0 1.0; visual mesh filename=package://robotiq_description/meshes/visual/hande/hand-e.dae scale=1.0 1.0 1.0
- added link hande_finger_distance_link
- added link hande_left_finger; collision box size=1.0 1.0 1.0; visual mesh filename=package://robotiq_description/meshes/visual/hande/left_fing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 scale=1.0 1.0 1.0
- added link hande_right_finger; collision box size=1.0 1.0 1.0; visual mesh filename=package://robotiq_description/meshes/visual/hande/right_fin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 scale=1.0 1.0 1.0
- added link tcp_link
Joints:
- added joint hande_finger_distance: type prismatic, parent hand_e_base_link, child hande_finger_distance_link, origin xyz=0 0 0.099 rpy=0 0 0, axis 1 0 0, limit lower=0.0 upper=0.05 effort=180 velocity=0.15
- added joint hande_left_finger_joint: type prismatic, parent hand_e_base_link, child hande_left_finger, origin xyz=0 0 0.099 rpy=0 0 0, axis -1 0 0, limit lower=0 upper=0.025 effort=180 velocity=0.15, mimic joint=hande_finger_distance multiplier=-0.5 offset=0.025
- added joint hande_right_finger_joint: type prismatic, parent hand_e_base_link, child hande_right_finger, origin xyz=0 0 0.099 rpy=0 0 0, axis 1 0 0, limit lower=0 upper=0.025 effort=180 velocity=0.15, mimic joint=hande_finger_distance multiplier=-0.5 offset=0.025
- added joint robotiq_hande_base_joint: type fixed, parent rv2fr_default_tcp, child hand_e_base_link, origin xyz=0 0 0 rpy=0 0 0
- added joint tcp_link_joint: type fixed, parent hand_e_base_link, child tcp_link, origin xyz=0 0 0.1325 rpy=0 0 -1.5707963267948966

Commit message: half woirking version for fortress.

File: melfa_description/urdf/rv2fr/rv2fr.urdf (robot description, URDF)
Before this commit: robot rv2fr, 14 links, 13 joints
Joints:
- joint hande_left_finger_joint: mimic joint=hande_finger_distance multiplier=-0.5 offset=0.025 -> (none)
- joint hande_right_finger_joint: mimic joint=hande_finger_distance multiplier=-0.5 offset=0.025 -> (none)

Commit message: Modify file to match jazzy

File: melfa_description/urdf/rv2fr/rv2fr.urdf (robot description, URDF)
Before this commit: robot rv2fr, 14 links, 13 joints
Links:
- link hand_e_base_link: geometry collision mesh filename=file://$(find robotiq_description)/meshes/collision/hande/h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 scale=1.0 1.0 1.0; visual mesh filename=file://$(find robotiq_description)/meshes/visual/hande/hand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 scale=1.0 1.0 1.0
- link hande_left_finger: geometry collision box size=1.0 1.0 1.0; visual mesh filename=file://$(find robotiq_description)/meshes/visual/hande/left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 scale=1.0 1.0 1.0
- link hande_right_finger: geometry collision box size=1.0 1.0 1.0; visual mesh filename=file://$(find robotiq_description)/meshes/visual/hande/righ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 scale=1.0 1.0 1.0
- link rv2fr_base: geometry collision mesh filename=file://$(find melfa_description)/meshes/rv2fr/base.STL; visual mesh filename=file://$(find melfa_description)/meshes/rv2fr/base.STL
- link rv2fr_elbow: geometry collision mesh filename=file://$(find melfa_description)/meshes/rv2fr/elbow.STL; visual mesh filename=file://$(find melfa_description)/meshes/rv2fr/elbow.STL
- link rv2fr_forearm: geometry collision mesh filename=file://$(find melfa_description)/meshes/rv2fr/forearm.STL; visual mesh filename=file://$(find melfa_description)/meshes/rv2fr/forearm.STL
- link rv2fr_hand_flange: geometry collision mesh filename=file://$(find melfa_description)/meshes/rv2fr/hand_flange.S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; visual mesh filename=file://$(find melfa_description)/meshes/rv2fr/hand_flange.S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
- link rv2fr_shoulder: geometry collision mesh filename=file://$(find melfa_description)/meshes/rv2fr/shoulder.STL; visual mesh filename=file://$(find melfa_description)/meshes/rv2fr/shoulder.STL
- link rv2fr_upper_arm: geometry collision mesh filename=file://$(find melfa_description)/meshes/rv2fr/upper_arm.STL; visual mesh filename=file://$(find melfa_description)/meshes/rv2fr/upper_arm.STL
- link rv2fr_wrist: geometry collision mesh filename=file://$(find melfa_description)/meshes/rv2fr/wrist.STL; visual mesh filename=file://$(find melfa_description)/meshes/rv2fr/wrist.STL
Joints:
- removed joint hande_left_finger_joint
- removed joint hande_right_finger_joint

File: melfa_description/urdf/rv2fr/rv2fr_macro.xacro (robot description, xacro)
@@ -87,11 +87,11 @@
             <origin rpy="0 0 0" xyz="0 0 0"/>
             <geometry>
-                <mesh filename="package://melfa_description/meshes/rv2fr/base.STL"/>
-            </geometry>
-            </visual>
-            <collision>
-            <origin rpy="0 0 0" xyz="0 0 0"/>
-            <geometry>
-                <mesh filename="package://melfa_description/meshes/rv2fr/base.STL"/>
+                <mesh filename="file://$(find melfa_description)/meshes/rv2fr/base.STL"/>
+            </geometry>
+            </visual>
+            <collision>
+            <origin rpy="0 0 0" xyz="0 0 0"/>
+            <geometry>
+                <mesh filename="file://$(find melfa_description)/meshes/rv2fr/base.STL"/>
             </geometry>
             </collision>
@@ -105,11 +105,11 @@
             <origin rpy="0 0 0" xyz="0 0 0"/>
             <geometry>
-                <mesh filename="package://melfa_description/meshes/rv2fr/shoulder.STL"/>
-            </geometry>
-            </visual>
-            <collision>
-            <origin rpy="0 0 0" xyz="0 0 0"/>
-            <geometry>
-                <mesh filename="package://melfa_description/meshes/rv2fr/shoulder.STL"/>
+                <mesh filename="file://$(find melfa_description)/meshes/rv2fr/shoulder.STL"/>
+            </geometry>
+            </visual>
+            <collision>
+            <origin rpy="0 0 0" xyz="0 0 0"/>
+            <geometry>
+                <mesh filename="file://$(find melfa_description)/meshes/rv2fr/shoulder.STL"/>
             </geometry>
             </collision>
@@ -123,11 +123,11 @@
             <origin rpy="0 0 0" xyz="0 0 0"/>
             <geometry>
-                <mesh filename="package://melfa_description/meshes/rv2fr/upper_arm.STL"/>
-            </geometry>
-            </visual>
-            <collision>
-            <origin rpy="0 0 0" xyz="0 0 0"/>
-            <geometry>
-                <mesh filename="package://melfa_description/meshes/rv2fr/upper_arm.STL"/>
+                <mesh filename="file://$(find melfa_description)/meshes/rv2fr/upper_arm.STL"/>
+            </geometry>
+            </visual>
+            <collision>
+            <origin rpy="0 0 0" xyz="0 0 0"/>
+            <geometry>
+                <mesh filename="file://$(find melfa_description)/meshes/rv2fr/upper_arm.STL"/>
             </geometry>
             </collision>
@@ -141,11 +141,11 @@
             <origin rpy="0 0 0" xyz="0 0 0"/>
             <geometry>
-                <mesh filename="package://melfa_description/meshes/rv2fr/elbow.STL"/>
-            </geometry>
-            </visual>
-            <collision>
-            <origin rpy="0 0 0" xyz="0 0 0"/>
-            <geometry>
-                <mesh filename="package://melfa_description/meshes/rv2fr/elbow.STL"/>
+                <mesh filename="file://$(find melfa_description)/meshes/rv2fr/elbow.STL"/>
+            </geometry>
+            </visual>
+            <collision>
+            <origin rpy="0 0 0" xyz="0 0 0"/>
+            <geometry>
+                <mesh filename="file://$(find melfa_description)/meshes/rv2fr/elbow.STL"/>
             </geometry>
             </collision>
@@ -159,11 +159,11 @@
             <origin rpy="0 0 0" xyz="0 0 0"/>
             <geometry>
-                <mesh filename="package://melfa_description/meshes/rv2fr/forearm.STL"/>
-            </geometry>
-            </visual>
-            <collision>
-            <origin rpy="0 0 0" xyz="0 0 0"/>
-            <geometry>
-                <mesh filename="package://melfa_description/meshes/rv2fr/forearm.STL"/>
+                <mesh filename="file://$(find melfa_description)/meshes/rv2fr/forearm.STL"/>
+            </geometry>
+            </visual>
+            <collision>
+            <origin rpy="0 0 0" xyz="0 0 0"/>
+            <geometry>
+                <mesh filename="file://$(find melfa_description)/meshes/rv2fr/forearm.STL"/>
             </geometry>
             </collision>
@@ -177,11 +177,11 @@
             <origin rpy="0 0 0" xyz="0 0 0"/>
             <geometry>
-                <mesh filename="package://melfa_description/meshes/rv2fr/wrist.STL"/>
-            </geometry>
-            </visual>
-            <collision>
-            <origin rpy="0 0 0" xyz="0 0 0"/>
-            <geometry>
-                <mesh filename="package://melfa_description/meshes/rv2fr/wrist.STL"/>
+                <mesh filename="file://$(find melfa_description)/meshes/rv2fr/wrist.STL"/>
+            </geometry>
+            </visual>
+            <collision>
+            <origin rpy="0 0 0" xyz="0 0 0"/>
+            <geometry>
+                <mesh filename="file://$(find melfa_description)/meshes/rv2fr/wrist.STL"/>
             </geometry>
             </collision>
@@ -195,11 +195,11 @@
             <origin rpy="0 0 0" xyz="0 0 0"/>
             <geometry>
-                <mesh filename="package://melfa_description/meshes/rv2fr/hand_flange.STL"/>
-            </geometry>
-            </visual>
-            <collision>
-            <origin rpy="0 0 0" xyz="0 0 0"/>
-            <geometry>
-                <mesh filename="package://melfa_description/meshes/rv2fr/hand_flange.STL"/>
+                <mesh filename="file://$(find melfa_description)/meshes/rv2fr/hand_flange.STL"/>
+            </geometry>
+            </visual>
+            <collision>
+            <origin rpy="0 0 0" xyz="0 0 0"/>
+            <geometry>
+                <mesh filename="file://$(find melfa_description)/meshes/rv2fr/hand_flange.STL"/>
             </geometry>
             </collision>

Commit message: Update urdf for moveit

File: melfa_description/urdf/rv2fr/rv2fr.urdf (robot description, URDF)
Before this commit: robot rv2fr, 14 links, 11 joints
Joints:
- added joint hande_left_finger_joint: type prismatic, parent hand_e_base_link, child hande_left_finger, origin xyz=0 0 0.099 rpy=0 0 0, axis -1 0 0, limit lower=0 upper=0.025 effort=180 velocity=0.08, mimic joint=hande_finger_distance multiplier=-0.5 offset=0.025
- added joint hande_right_finger_joint: type prismatic, parent hand_e_base_link, child hande_right_finger, origin xyz=0 0 0.099 rpy=0 0 0, axis 1 0 0, limit lower=0 upper=0.025 effort=180 velocity=0.08, mimic joint=hande_finger_distance multiplier=-0.5 offset=0.025
