Commit message: Moveit config (#1)
* WIP commit to create moveit_config

* Update srdf to use different tiip link

* update moveit config

* Migrate from _gripper postfix to directly use rv2fr

* Remove comments.

* Update configs for moveit pkg.

---------

Co-authored-by: NinjaDev108 <jsshankar@gmail.com>

File: melfa_moveit_config/melfa_rv2fr_moveit_config/config/rv2fr.ros2_control.xacro (robot description, xacro)
@@ -50,4 +50,12 @@
                 <state_interface name="velocity"/>
             </joint>
+            <!-- Robotiq Hand-E Gripper Joint -->
+            <joint name="hande_finger_distance">
+                <command_interface name="position"/>
+                <state_interface name="position">
+                    <param name="initial_value">0.0</param>
+                </state_interface>
+                <state_interface name="velocity"/>
+            </joint>
         </ros2_control>
     </xacro:macro>
